File: hardware/pot8/umodular_pot8.brd (EAGLE design)
At the start: 199.5 x 25 mm, 17 parts, among them IC1 4051N

Commit message: Fix module Pot8 size to fixed 10x2.5cm
Other:
- board size 199.5 x 25 mm -> 200 x 25 mm
- board text added: "uMODULAR Pot8 rev. 0.2 CC-BY-SA 4 - Romulo Silva http://midilab.co"
- board text removed: "uMODULAR Pot8 rev. 0.1 CC-BY-SA 4 - Romulo Silva http://midilab.co"
Changed lines of the file:
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@@
 <board>
 <plain>
-<wire x1="0.5" y1="0" x2="200" y2="0" width="0" layer="20"/>
+<wire x1="0" y1="0" x2="200" y2="0" width="0" layer="20"/>
 <wire x1="200" y1="0" x2="200" y2="25" width="0" layer="20"/>
-<wire x1="200" y1="25" x2="0.5" y2="25" width="0" layer="20"/>
-<wire x1="0.5" y1="25" x2="0.5" y2="0" width="0" layer="20"/>
-<text x="109.875" y="19.625" size="1.6764" layer="25" font="fixed">     uMODULAR Pot8 rev. 0.1
+<wire x1="200" y1="25" x2="0" y2="25" width="0" layer="20"/>
+<wire x1="0" y1="25" x2="0" y2="0" width="0" layer="20"/>
+<text x="109.875" y="19.625" size="1.6764" layer="25" font="fixed">     uMODULAR Pot8 rev. 0.2
      CC-BY-SA 4 - Romulo Silva http://midilab.co</text>
-<text x="190.125" y="19.625" size="1.6764" layer="16" font="fixed" rot="MR0">     uMODULAR Pot8 rev. 0.1
+<text x="190.125" y="19.625" size="1.6764" layer="16" font="fixed" rot="MR0">     uMODULAR Pot8 rev. 0.2
      CC-BY-SA 4 - Romulo Silva http://midilab.co</text>
 </plain>
