File: hardware/fader8/umodular_fader8.brd (EAGLE design)
At the start: 200 x 80 mm, 21 parts, among them IC1 4051N

Commit message: Fix module Fader8 size to fixed 20x8cm
Parts:
- U$10: device SparkFun-Aesthetics2:OSHW-LOGO-M -> SparkFun-Aesthetics3:OSHW-LOGO-M
Other:
- board text added: "uMODULAR Fader8 rev. 0.2 CC-BY-SA - Romulo Silva http://midilab.co"
- board text removed: "uMODULAR Fader8 rev. 0.1 CC-BY-SA - Romulo Silva http://midilab.co"
Changed lines of the file:
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@@
 <board>
 <plain>
-<wire x1="0" y1="0" x2="199.98" y2="0" width="0" layer="20"/>
-<wire x1="199.98" y1="0" x2="199.98" y2="80" width="0" layer="20"/>
-<wire x1="199.98" y1="80" x2="0" y2="80" width="0" layer="20"/>
+<wire x1="0" y1="0" x2="200" y2="0" width="0" layer="20"/>
+<wire x1="200" y1="0" x2="200" y2="80" width="0" layer="20"/>
+<wire x1="200" y1="80" x2="0" y2="80" width="0" layer="20"/>
 <wire x1="0" y1="80" x2="0" y2="0" width="0" layer="20"/>
-<text x="1.75" y="59" size="1.4224" layer="27" font="vector" rot="R270">uMODULAR Fader8 rev. 0.1
+<text x="1.75" y="59" size="1.4224" layer="27" font="vector" rot="R270">uMODULAR Fader8 rev. 0.2
 CC-BY-SA - Romulo Silva http://midilab.co</text>
-<text x="198" y="59" size="1.4224" layer="26" font="vector" rot="MR270">uMODULAR Fader8 rev. 0.1
+<text x="198" y="59" size="1.4224" layer="16" font="vector" rot="MR270">uMODULAR Fader8 rev. 0.2
 CC-BY-SA - Romulo Silva http://midilab.co</text>
 </plain>
@@
 <element name="U$8" library="holes" package="3,0" value="" x="125" y="12.5"/>
 <element name="U$9" library="SparkFun-Aesthetics" package="OSHW-LOGO-M" value="" x="3.75" y="5.75"/>
-<element name="U$10" library="SparkFun-Aesthetics2" package="OSHW-LOGO-M" value="" x="196.25" y="5.75"/>
+<element name="U$10" library="SparkFun-Aesthetics3" package="OSHW-LOGO-M" value="" x="196.25" y="5.75"/>
 </elements>
 <signals>
