File: ctrl16/umodular_ctrl16.brd (EAGLE design)
At the start: 100 x 125 mm, 73 parts, among them IC1 4051N, IC2 4051N, IC3 74HC595N, IC4 74HC165N

Commit message: ctrl16 revision 0.1
Parts:
- removed R92, R93, R94, R95, R96, R97: 10k, resistor:0204/7
- added R1, R4, R5, R6, R7: 220, rcl:0204/7
- added R9: 10k, resistor:0204/7
- R12, R13, R14, R15, R16, R17: value 220 -> 10k; device rcl:0204/7 -> resistor:0204/7
- R3: value 10k -> 220; device resistor:0204/7 -> rcl:0204/7
- moved R13 52.2 mm to (12.5, 8.76), turned to 0 degrees
- moved R17 50.8 mm to (12.5, 20.7), turned to 0 degrees
- moved R15 50.8 mm to (62.5, 20.7), turned to 0 degrees
- moved R3 25.1 mm to (62.5, 23.8)
- moved R2 25.0 mm to (37.5, 23.8)
- moved C1 23.5 mm to (49.8, 92.8)
- moved C2 23.5 mm to (50.0, 116.3)
- moved R12 15.1 mm to (37.5, 8.70), turned to 0 degrees
- moved R16 8.96 mm to (37.5, 20.7), turned to 0 degrees
- moved R14 3.04 mm to (87.5, 20.7), turned to 0 degrees
- renumbered C14 to C3, C5 to C4, R18 to R8, R98 to R11, R99 to R10
Connections:
- net N$2: now also R17.2; no longer R92.2
- net N$3: now also R16.2; no longer R93.2
- net N$4: now also R15.2; no longer R94.2
- net N$5: now also R14.2; no longer R95.2
- net N$6: now also R13.2; no longer R96.2
- net N$7: now also R12.2; no longer R97.2
- net N$76: now also R7.1; no longer R17.1
- net N$77: now also R6.1; no longer R16.1
- net N$78: now also R5.1; no longer R15.1
- net N$79: now also R4.1; no longer R14.1
- net N$80: now also R3.1; no longer R13.1
- net N$81: now also R2.1; no longer R12.1
- net N$82: now also R1.1; no longer R2.1
- net N$83: now also R1.2; no longer R2.2
- net N$84: now also R2.2; no longer R12.2
- net N$85: now also R4.2; no longer R14.2
- net N$86: now also R3.2; no longer R13.2
- net N$87: now also R5.2; no longer R15.2
- net N$88: now also R6.2; no longer R16.2
- net N$89: now also R7.2; no longer R17.2
- net SPI_MISO_CHAIN: now also R9.1; no longer R3.1
- net VCC: now also R12.1, R13.1, R14.1, R15.1, R16.1, R17.1, R9.2; no longer R3.2, R92.1, R93.1, R94.1, R95.1, R96.1, R97.1
