File: pot16/umodular_pot16.brd (EAGLE design)
At the start: 100 x 100 mm, 32 parts, among them IC1 4051N, IC2 4051N

Commit message: pot16 revision 01
Parts:
- moved C1 23.5 mm to (49.8, 67.8)
- moved C2 23.5 mm to (50.0, 91.3)
Changed lines of the file:
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@@
 <attribute name="VALUE" x="50.685" y="82.103" size="1.27" layer="28" ratio="10" rot="MR270"/>
 </element>
-<element name="C1" library="rcl" package="C050-024X044" value="100 nF" x="49.96" y="91.28" smashed="yes" rot="MR180">
+<element name="C2" library="rcl" package="C050-024X044" value="100 nF" x="49.96" y="91.28" smashed="yes" rot="MR180">
 <attribute name="NAME" x="53.471" y="91.913" size="1.27" layer="26" ratio="10" rot="MR180"/>
 <attribute name="VALUE" x="40.251" y="91.777" size="1.27" layer="28" ratio="10" rot="MR180"/>
@@
 <attribute name="VALUE" x="50.745" y="58.523" size="1.27" layer="28" ratio="10" rot="MR270"/>
 </element>
-<element name="C2" library="rcl" package="C050-024X044" value="100 nF" x="49.81" y="67.77" smashed="yes" rot="MR180">
+<element name="C1" library="rcl" package="C050-024X044" value="100 nF" x="49.81" y="67.77" smashed="yes" rot="MR180">
 <attribute name="NAME" x="53.541" y="68.393" size="1.27" layer="26" ratio="10" rot="MR180"/>
 <attribute name="VALUE" x="39.501" y="68.337" size="1.27" layer="28" ratio="10" rot="MR180"/>
@@
 <contactref element="ANALOG_2" pad="9"/>
 <contactref element="IC2" pad="16"/>
-<contactref element="C1" pad="1"/>
+<contactref element="C2" pad="1"/>
 <contactref element="POT_16" pad="P$3"/>
 <contactref element="POT_15" pad="P$3"/>
@@
 <contactref element="POT_2" pad="P$3"/>
 <contactref element="POT_1" pad="P$3"/>
-<contactref element="C2" pad="1"/>
+<contactref element="C1" pad="1"/>
 <wire x1="67.58" y1="49.87" x2="67.63" y2="49.87" width="0.8128" layer="1"/>
 <wire x1="67.63" y1="49.87" x2="69.59" y2="47.91" width="0.8128" layer="1"/>
@@
 <contactref element="POT_15" pad="P$1"/>
 <contactref element="POT_14" pad="P$1"/>
-<contactref element="C1" pad="2"/>
+<contactref element="C2" pad="2"/>
 <contactref element="IC2" pad="7"/>
 <contactref element="IC2" pad="8"/>
@@
 <contactref element="POT_2" pad="P$1"/>
 <contactref element="POT_1" pad="P$1"/>
-<contactref element="C2" pad="2"/>
+<contactref element="C1" pad="2"/>
 <contactref element="IC1" pad="7"/>
 <contactref element="IC1" pad="8"/>
