File: mix4/umodular_mix4.brd (EAGLE design)
At the start: 100 x 125 mm, 62 parts, among them IC1 4051N, IC11 74HC165N, IC22 74HC595N

Commit message: mix4 revision 01
Parts:
- removed R92, R93, R94, R95, R96, R97: 10k, resistor:0204/7
- added R1, R4, R5, R6, R7: 220, rcl:0204/7
- added R9: 10k, resistor:0204/7
- R12, R13, R14, R15, R16, R17: value 220 -> 10k; device rcl:0204/7 -> resistor:0204/7
- R3: value 10k -> 220; device resistor:0204/7 -> rcl:0204/7
- moved R13 52.2 mm to (12.5, 8.76), turned to 0 degrees
- moved R17 50.8 mm to (12.5, 20.7), turned to 0 degrees
- moved R15 50.8 mm to (62.5, 20.7), turned to 0 degrees
- moved R3 25.1 mm to (62.5, 23.8)
- moved R2 25.0 mm to (37.5, 23.8)
- moved R12 15.1 mm to (37.5, 8.70), turned to 0 degrees
- moved R16 8.96 mm to (37.5, 20.7), turned to 0 degrees
- moved R14 3.04 mm to (87.5, 20.7), turned to 0 degrees
- renumbered C14 to C2, C5 to C3, R18 to R8, R98 to R11, R99 to R10
Connections:
- net N$2: now also R17.2; no longer R92.2
- net N$3: now also R16.2; no longer R93.2
- net N$4: now also R15.2; no longer R94.2
- net N$5: now also R14.2; no longer R95.2
- net N$6: now also R13.2; no longer R96.2
- net N$7: now also R12.2; no longer R97.2
- net N$76: now also R7.1; no longer R17.1
- net N$77: now also R6.1; no longer R16.1
- net N$78: now also R5.1; no longer R15.1
- net N$79: now also R4.1; no longer R14.1
- net N$80: now also R3.1; no longer R13.1
- net N$81: now also R2.1; no longer R12.1
- net N$82: now also R1.1; no longer R2.1
- net N$83: now also R1.2; no longer R2.2
- net N$84: now also R2.2; no longer R12.2
- net N$85: now also R4.2; no longer R14.2
- net N$86: now also R3.2; no longer R13.2
- net N$87: now also R5.2; no longer R15.2
- net N$88: now also R6.2; no longer R16.2
- net N$89: now also R7.2; no longer R17.2
- net SPI_MISO_CHAIN: now also R9.1; no longer R3.1
- net VCC: now also R12.1, R13.1, R14.1, R15.1, R16.1, R17.1, R9.2; no longer R3.2, R92.1, R93.1, R94.1, R95.1, R96.1, R97.1

Commit message: fix bounrs fader part. swaped pin 2 and 1.
Connections:
- net N$274: now also FADER_1.2; no longer FADER_1.2A
- net N$275: now also FADER_2.2; no longer FADER_2.2A
- net N$276: now also FADER_3.2; no longer FADER_3.2A
- net N$277: now also FADER_4.2; no longer FADER_4.2A
Routing:
- net AGND: track 439.1 -> 441.7 mm, vias 1 -> 3
- net N$275: track 82.0 -> 83.4 mm
- net N$277: track 97.8 -> 99.2 mm
- net N$274: track 91.2 -> 92.4 mm
- net N$276: track 87.8 -> 87.7 mm, vias 0 -> 1
Changed lines of the file:
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@@
 <signal name="N$274">
 <contactref element="IC1" pad="13"/>
-<contactref element="FADER_1" pad="2A"/>
+<contactref element="FADER_1" pad="2"/>
 <wire x1="46.19" y1="99.97" x2="43.4" y2="99.97" width="0.4064" layer="16"/>
 <wire x1="43.4" y1="99.97" x2="37.5" y2="94.07" width="0.4064" layer="16"/>
@@
 <wire x1="26.7" y1="52.05" x2="18.41" y2="43.76" width="0.4064" layer="1"/>
 <via x="18.41" y="43.76" extent="1-16" drill="0.6" shape="square"/>
-<wire x1="18.41" y1="43.76" x2="18.41" y2="37.08" width="0.4064" layer="16"/>
-<wire x1="18.41" y1="37.08" x2="10.72" y2="29.39" width="0.4064" layer="16"/>
-<wire x1="10.72" y1="29.39" x2="10.72" y2="25.78" width="0.4064" layer="16"/>
-<wire x1="10.72" y1="25.78" x2="10.75" y2="25.75" width="0.4064" layer="16"/>
+<wire x1="18.41" y1="43.76" x2="18.41" y2="32.59" width="0.4064" layer="16"/>
+<wire x1="18.41" y1="32.59" x2="19.29" y2="31.71" width="0.4064" layer="16"/>
+<wire x1="19.29" y1="31.71" x2="19.29" y2="27.53" width="0.4064" layer="16"/>
+<wire x1="19.29" y1="27.53" x2="17.49" y2="25.73" width="0.4064" layer="16"/>
+<wire x1="17.49" y1="25.73" x2="14.27" y2="25.73" width="0.4064" layer="16"/>
+<wire x1="14.27" y1="25.73" x2="14.25" y2="25.75" width="0.4064" layer="16"/>
 </signal>
 <signal name="N$275">
 <contactref element="IC1" pad="14"/>
-<contactref element="FADER_2" pad="2A"/>
+<contactref element="FADER_2" pad="2"/>
 <wire x1="46.19" y1="102.51" x2="44.6" y2="102.51" width="0.4064" layer="1"/>
 <wire x1="44.6" y1="102.51" x2="35.87" y2="93.78" width="0.4064" layer="1"/>
@@
 <wire x1="35.8" y1="50.96" x2="35.83" y2="50.93" width="0.4064" layer="1"/>
 <via x="35.83" y="50.93" extent="1-16" drill="0.6" shape="square"/>
-<wire x1="35.83" y1="50.93" x2="35.83" y2="29.47" width="0.4064" layer="16"/>
-<wire x1="35.83" y1="29.47" x2="35.76" y2="29.4" width="0.4064" layer="16"/>
-<via x="35.76" y="29.4" extent="1-16" drill="0.6" shape="square"/>
-<wire x1="35.76" y1="29.4" x2="35.76" y2="25.76" width="0.4064" layer="1"/>
-<wire x1="35.76" y1="25.76" x2="35.75" y2="25.75" width="0.4064" layer="1"/>
+<wire x1="35.83" y1="50.93" x2="35.83" y2="31.98" width="0.4064" layer="16"/>
+<wire x1="35.83" y1="31.98" x2="38.52" y2="29.29" width="0.4064" layer="16"/>
+<via x="38.52" y="29.29" extent="1-16" drill="0.6" shape="square"/>
+<wire x1="38.52" y1="29.29" x2="38.52" y2="26.48" width="0.4064" layer="1"/>
+<wire x1="38.52" y1="26.48" x2="39.25" y2="25.75" width="0.4064" layer="1"/>
 </signal>
 <signal name="N$276">
 <contactref element="IC1" pad="15"/>
-<contactref element="FADER_3" pad="2A"/>
+<contactref element="FADER_3" pad="2"/>
 <wire x1="46.19" y1="105.05" x2="47.63" y2="105.05" width="0.4064" layer="16"/>
 <wire x1="47.63" y1="105.05" x2="49.15" y2="103.53" width="0.4064" layer="16"/>
@@
 <wire x1="49.15" y1="95.86" x2="51.46" y2="93.55" width="0.4064" layer="16"/>
 <wire x1="51.46" y1="93.55" x2="51.46" y2="88.17" width="0.4064" layer="16"/>
-<wire x1="51.46" y1="88.17" x2="62.74" y2="76.89" width="0.4064" layer="16"/>
-<wire x1="62.74" y1="76.89" x2="62.74" y2="27.74" width="0.4064" layer="16"/>
-<wire x1="62.74" y1="27.74" x2="60.75" y2="25.75" width="0.4064" layer="16"/>
+<wire x1="51.46" y1="88.17" x2="62.75" y2="76.88" width="0.4064" layer="16"/>
+<wire x1="64.25" y1="25.75" x2="64.14" y2="25.75" width="0.4064" layer="1"/>
+<wire x1="64.14" y1="25.75" x2="62.75" y2="27.14" width="0.4064" layer="1"/>
+<wire x1="62.75" y1="27.14" x2="62.75" y2="30.26" width="0.4064" layer="1"/>
+<via x="62.75" y="30.26" extent="1-16" drill="0.6" shape="square"/>
+<wire x1="62.75" y1="30.26" x2="62.75" y2="76.88" width="0.4064" layer="16"/>
 </signal>
 <signal name="N$277">
 <contactref element="IC1" pad="12"/>
-<contactref element="FADER_4" pad="2A"/>
+<contactref element="FADER_4" pad="2"/>
 <wire x1="46.19" y1="97.43" x2="47.3" y2="97.43" width="0.4064" layer="16"/>
 <wire x1="47.3" y1="97.43" x2="48.16" y2="96.57" width="0.4064" layer="16"/>
@@
 <wire x1="60.08" y1="76.94" x2="75.47" y2="76.94" width="0.4064" layer="1"/>
 <wire x1="75.47" y1="76.94" x2="85.85" y2="66.56" width="0.4064" layer="1"/>
-<wire x1="85.85" y1="66.56" x2="85.85" y2="25.85" width="0.4064" layer="1"/>
-<wire x1="85.85" y1="25.85" x2="85.75" y2="25.75" width="0.4064" layer="1"/>
+<wire x1="85.85" y1="66.56" x2="85.89" y2="29.55" width="0.4064" layer="1"/>
+<wire x1="85.89" y1="29.55" x2="85.89" y2="29.11" width="0.4064" layer="1"/>
+<wire x1="85.89" y1="29.11" x2="89.25" y2="25.75" width="0.4064" layer="1"/>
 </signal>
 <signal name="N$278">
@@
 <wire x1="11.12" y1="107.64" x2="11.12" y2="116.12" width="0.8128" layer="16"/>
 <wire x1="11.12" y1="116.12" x2="9.6" y2="117.64" width="0.8128" layer="16"/>
-<wire x1="89.25" y1="25.75" x2="93.55" y2="25.75" width="0.8128" layer="16"/>
-<wire x1="93.55" y1="25.75" x2="98.64" y2="30.84" width="0.8128" layer="16"/>
-<wire x1="98.64" y1="30.84" x2="98.64" y2="110.97" width="0.8128" layer="16"/>
+<wire x1="98.64" y1="30.59" x2="98.64" y2="110.97" width="0.8128" layer="16"/>
 <wire x1="98.64" y1="110.97" x2="98.65" y2="110.98" width="0.8128" layer="16"/>
-<wire x1="14.25" y1="25.75" x2="14.25" y2="26.98" width="0.8128" layer="16"/>
-<wire x1="14.25" y1="26.98" x2="14.99" y2="27.72" width="0.8128" layer="16"/>
-<wire x1="14.99" y1="27.72" x2="38.31" y2="27.72" width="0.8128" layer="16"/>
-<wire x1="38.31" y1="27.72" x2="39.25" y2="26.78" width="0.8128" layer="16"/>
-<wire x1="39.25" y1="26.78" x2="39.25" y2="25.75" width="0.8128" layer="16"/>
-<wire x1="39.25" y1="25.75" x2="39.25" y2="26.76" width="0.8128" layer="1"/>
-<wire x1="39.25" y1="26.76" x2="40.19" y2="27.7" width="0.8128" layer="1"/>
-<wire x1="40.19" y1="27.7" x2="63.27" y2="27.7" width="0.8128" layer="1"/>
-<wire x1="63.27" y1="27.7" x2="64.31" y2="26.66" width="0.8128" layer="1"/>
-<wire x1="64.31" y1="26.66" x2="64.31" y2="25.81" width="0.8128" layer="1"/>
-<wire x1="64.31" y1="25.81" x2="64.25" y2="25.75" width="0.8128" layer="1"/>
-<wire x1="64.25" y1="25.75" x2="64.25" y2="26.73" width="0.8128" layer="16"/>
-<wire x1="64.25" y1="26.73" x2="65.27" y2="27.75" width="0.8128" layer="16"/>
-<wire x1="65.27" y1="27.75" x2="88.26" y2="27.75" width="0.8128" layer="16"/>
-<wire x1="88.26" y1="27.75" x2="89.26" y2="26.75" width="0.8128" layer="16"/>
-<wire x1="89.26" y1="26.75" x2="89.26" y2="25.76" width="0.8128" layer="16"/>
-<wire x1="89.26" y1="25.76" x2="89.25" y2="25.75" width="0.8128" layer="16"/>
 <wire x1="53.81" y1="94.89" x2="53.81" y2="92.35" width="0.8128" layer="16"/>
 <wire x1="53.81" y1="92.35" x2="53.81" y2="89.81" width="0.8128" layer="16"/>
+<wire x1="98.64" y1="30.59" x2="95.73" y2="27.68" width="0.8128" layer="16"/>
+<wire x1="95.73" y1="27.68" x2="87.68" y2="27.68" width="0.8128" layer="16"/>
+<wire x1="87.68" y1="27.68" x2="85.75" y2="25.75" width="0.8128" layer="16"/>
+<wire x1="60.18" y1="27.7" x2="60.72" y2="27.16" width="0.8128" layer="1"/>
+<wire x1="60.72" y1="27.16" x2="60.72" y2="25.78" width="0.8128" layer="1"/>
+<wire x1="60.72" y1="25.78" x2="60.75" y2="25.75" width="0.8128" layer="1"/>
+<wire x1="10.75" y1="25.75" x2="10.75" y2="25.78" width="0.8128" layer="1"/>
+<wire x1="10.75" y1="25.78" x2="12.72" y2="27.75" width="0.8128" layer="1"/>
+<wire x1="85.75" y1="25.75" x2="85.7" y2="25.75" width="0.8128" layer="16"/>
+<wire x1="85.7" y1="25.75" x2="83.72" y2="27.73" width="0.8128" layer="16"/>
+<wire x1="83.72" y1="27.73" x2="62.73" y2="27.73" width="0.8128" layer="16"/>
+<wire x1="62.73" y1="27.73" x2="60.75" y2="25.75" width="0.8128" layer="16"/>
+<wire x1="12.72" y1="27.75" x2="24.46" y2="27.75" width="0.8128" layer="1"/>
+<wire x1="24.46" y1="27.75" x2="24.5" y2="27.79" width="0.8128" layer="1"/>
+<via x="24.5" y="27.79" extent="1-16" drill="0.6" shape="square"/>
+<wire x1="24.5" y1="27.79" x2="34.83" y2="27.79" width="0.8128" layer="16"/>
+<wire x1="34.83" y1="27.79" x2="35.7" y2="26.92" width="0.8128" layer="16"/>
+<wire x1="35.7" y1="26.92" x2="35.75" y2="26.87" width="0.8128" layer="16"/>
+<wire x1="35.75" y1="26.87" x2="35.75" y2="25.75" width="0.8128" layer="16"/>
+<wire x1="60.18" y1="27.7" x2="44.91" y2="27.7" width="0.8128" layer="1"/>
+<wire x1="44.91" y1="27.7" x2="43.23" y2="26.02" width="0.8128" layer="1"/>
+<via x="43.23" y="26.02" extent="1-16" drill="0.6" shape="square"/>
+<wire x1="43.23" y1="26.02" x2="42.4" y2="26.02" width="0.8128" layer="16"/>
+<wire x1="42.4" y1="26.02" x2="40.54" y2="27.88" width="0.8128" layer="16"/>
+<wire x1="40.54" y1="27.88" x2="36.66" y2="27.88" width="0.8128" layer="16"/>
+<wire x1="36.66" y1="27.88" x2="35.7" y2="26.92" width="0.8128" layer="16"/>
 </signal>
 </signals>
