File: mix4/umodular_mix4.sch (EAGLE design)
At the start: 50 parts, among them IC1 4051N, IC11 74HC165N, IC22 74HC595N

Commit message: mix4 revision 01
Parts:
- removed R92, R93, R94, R95, R96, R97: 10k, resistor:R-US_0204/7
- added R1, R4, R5, R6, R7: 220, rcl:R-US_0204/7
- added R9: 10k, resistor:R-US_0204/7
- R12, R13, R14, R15, R16, R17: value 220 -> 10k; device rcl:R-US_0204/7 -> resistor:R-US_0204/7
- R3: value 10k -> 220; device resistor:R-US_0204/7 -> rcl:R-US_0204/7
- renumbered C14 to C2, C5 to C3, R18 to R8, R98 to R11, R99 to R10
Connections:
- net N$2: now also R17.2; no longer R92.2
- net N$3: now also R16.2; no longer R93.2
- net N$4: now also R15.2; no longer R94.2
- net N$5: now also R14.2; no longer R95.2
- net N$6: now also R13.2; no longer R96.2
- net N$7: now also R12.2; no longer R97.2
- net N$76: now also R7.1; no longer R17.1
- net N$77: now also R6.1; no longer R16.1
- net N$78: now also R5.1; no longer R15.1
- net N$79: now also R4.1; no longer R14.1
- net N$80: now also R3.1; no longer R13.1
- net N$81: now also R2.1; no longer R12.1
- net N$82: now also R1.1; no longer R2.1
- net N$83: now also R1.2; no longer R2.2
- net N$84: now also R2.2; no longer R12.2
- net N$85: now also R4.2; no longer R14.2
- net N$86: now also R3.2; no longer R13.2
- net N$87: now also R5.2; no longer R15.2
- net N$88: now also R6.2; no longer R16.2
- net N$89: now also R7.2; no longer R17.2
- net SPI_MISO_CHAIN: now also R9.1; no longer R3.1
- net VCC: now also R12.1, R13.1, R14.1, R15.1, R16.1, R17.1, R9.2; no longer R3.2, R92.1, R93.1, R94.1, R95.1, R96.1, R97.1
Other:
- moved on the sheet: R12, R13, R14, R15, R16, R17, R2, R3

Commit message: fix bounrs fader part. swaped pin 2 and 1.
Connections:
- net AGND: now also FADER_1.1, FADER_2.1, FADER_3.1, FADER_4.1; no longer FADER_1.E, FADER_2.E, FADER_3.E, FADER_4.E
- net N$274: now also FADER_1.2; no longer FADER_1.S
- net N$275: now also FADER_2.2; no longer FADER_2.S
- net N$276: now also FADER_3.2; no longer FADER_3.S
- net N$277: now also FADER_4.2; no longer FADER_4.S
- net VCC: now also FADER_1.3, FADER_2.3, FADER_3.3, FADER_4.3; no longer FADER_1.A, FADER_2.A, FADER_3.A, FADER_4.A
Changed lines of the file:
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@@
 <segment>
 <label x="381" y="172.72" size="1.778" layer="95" rot="R270"/>
-<pinref part="FADER_1" gate="G$1" pin="A"/>
+<pinref part="FADER_1" gate="G$1" pin="3"/>
 <wire x1="381" y1="231.14" x2="381" y2="223.52" width="0.1524" layer="91"/>
 <wire x1="381" y1="223.52" x2="381" y2="215.9" width="0.1524" layer="91"/>
@@
 <wire x1="381" y1="177.8" x2="381" y2="170.18" width="0.1524" layer="91"/>
 <junction x="381" y="177.8"/>
-<pinref part="FADER_2" gate="G$1" pin="A"/>
+<pinref part="FADER_2" gate="G$1" pin="3"/>
 <junction x="381" y="185.42"/>
-<pinref part="FADER_3" gate="G$1" pin="A"/>
+<pinref part="FADER_3" gate="G$1" pin="3"/>
 <junction x="381" y="193.04"/>
-<pinref part="FADER_4" gate="G$1" pin="A"/>
+<pinref part="FADER_4" gate="G$1" pin="3"/>
 <junction x="381" y="200.66"/>
 <pinref part="POT_4" gate="G$1" pin="A"/>
@@
 <wire x1="373.38" y1="182.88" x2="317.5" y2="198.12" width="0.1524" layer="91"/>
 <pinref part="IC1" gate="A" pin="X0"/>
-<pinref part="FADER_1" gate="G$1" pin="S"/>
+<pinref part="FADER_1" gate="G$1" pin="2"/>
 </segment>
 </net>
@@
 <wire x1="373.38" y1="190.5" x2="317.5" y2="200.66" width="0.1524" layer="91"/>
 <pinref part="IC1" gate="A" pin="X1"/>
-<pinref part="FADER_2" gate="G$1" pin="S"/>
+<pinref part="FADER_2" gate="G$1" pin="2"/>
 </segment>
 </net>
@@
 <wire x1="373.38" y1="198.12" x2="317.5" y2="203.2" width="0.1524" layer="91"/>
 <pinref part="IC1" gate="A" pin="X2"/>
-<pinref part="FADER_3" gate="G$1" pin="S"/>
+<pinref part="FADER_3" gate="G$1" pin="2"/>
 </segment>
 </net>
@@
 <wire x1="373.38" y1="205.74" x2="317.5" y2="205.74" width="0.1524" layer="91"/>
 <pinref part="IC1" gate="A" pin="X3"/>
-<pinref part="FADER_4" gate="G$1" pin="S"/>
+<pinref part="FADER_4" gate="G$1" pin="2"/>
 </segment>
 </net>
@@
 <segment>
 <label x="365.76" y="172.72" size="1.778" layer="95" rot="R270"/>
-<pinref part="FADER_1" gate="G$1" pin="E"/>
+<pinref part="FADER_1" gate="G$1" pin="1"/>
 <wire x1="365.76" y1="231.14" x2="365.76" y2="223.52" width="0.1524" layer="91"/>
 <wire x1="365.76" y1="223.52" x2="365.76" y2="215.9" width="0.1524" layer="91"/>
@@
 <wire x1="365.76" y1="177.8" x2="365.76" y2="170.18" width="0.1524" layer="91"/>
 <junction x="365.76" y="177.8"/>
-<pinref part="FADER_2" gate="G$1" pin="E"/>
+<pinref part="FADER_2" gate="G$1" pin="1"/>
 <junction x="365.76" y="185.42"/>
-<pinref part="FADER_3" gate="G$1" pin="E"/>
+<pinref part="FADER_3" gate="G$1" pin="1"/>
 <junction x="365.76" y="193.04"/>
-<pinref part="FADER_4" gate="G$1" pin="E"/>
+<pinref part="FADER_4" gate="G$1" pin="1"/>
 <junction x="365.76" y="200.66"/>
 <pinref part="POT_4" gate="G$1" pin="E"/>
